Commit message: final

File: urdf/gazebo_control.xacro (robot description, xacro)
@@ -3,15 +3,12 @@
     <gazebo>
         <plugin name="diff_drive" filename="libgazebo_ros_diff_drive.so">
-            <!-- Wheel Information -->
             <left_joint>r_joint</left_joint>
             <right_joint>lf_joint</right_joint>
             <wheel_separation>0.59808</wheel_separation>
             <wheel_diameter>0.08</wheel_diameter>
-            <!-- Limits -->
             <max_wheel_torque>200</max_wheel_torque>
             <max_wheel_acceleration>10.0</max_wheel_acceleration>
-            <!-- Output -->
             <odometry_frame>odom</odometry_frame>
-            <robot_base_frame>base</robot_base_frame>
+            <robot_base_frame>base_link</robot_base_frame>
             <publish_odom>true</publish_odom>
             <publish_odom_tf>true</publish_odom_tf>
@@ -19,3 +16,37 @@
         </plugin>
     </gazebo>
+    <gazebo reference="base_link">
+        <material>Gazebo/Black</material>
+    </gazebo>
+     <gazebo reference="caster">
+        <material>Gazebo/Green</material>
+    </gazebo>
+     <gazebo reference="wc">
+        <material>Gazebo/Orange</material>
+        <mu1 value="0.001"/>
+        <mu2 value="0.001"/>
+    </gazebo>
+     <gazebo reference="l_wheel">
+        <material>Gazebo/Blue</material>
+    </gazebo>
+     <gazebo reference="r_wheel">
+        <material>Gazebo/Blue</material>
+    </gazebo>
+    <gazebo>
+        <plugin name="gazebo_ros_joint_state_publisher"
+            filename="libgazebo_ros_joint_state_publisher.so">
+            <update_rate>20</update_rate>
+            <joint_name>lf_joint</joint_name>
+            <joint_name>r_joint</joint_name>
+            <joint_name>caster_joint</joint_name>
+            <joint_name>wc_joint</joint_name>
+            <joint_name>base_joint</joint_name>
+        </plugin>
+    </gazebo>
+    <gazebo>
+        <plugin name="gazebo_ros_joint_pose_trajectory"
+            filename="libgazebo_ros_joint_pose_trajectory.so">
+            <update_rate>20</update_rate>
+        </plugin>
+    </gazebo>
 </robot>

File: urdf/robot_.xacro (robot description, xacro)
@@ -19,18 +19,4 @@
     <!-- include all the contents of example_include.xacro first. Go check it out! -->
     <xacro:include filename="example_include.xacro" />
-    <!-- edit and add base link ... this can handel from solidworks instead of here -->
-  <link name="base">
-  </link>
-  <joint
-    name="base_joint"
-    type="fixed">
-    <origin
-      xyz="0.18435 0 -9.1429E-05"
-      rpy="0 0 0" />
-    <parent
-      link="base" />
-    <child
-      link="base_link" />
-  </joint>
   <link
     name="base_link">
@@ -321,5 +307,5 @@
           filename="file://$(find test_robot)/meshes/wc.STL" />
         -->
-        <cylinder radius="0.05" length ="0.024" />
+        <cylinder radius="0.025" length ="0.024" />
       </geometry>
     </collision>
